Commit message: Just got through the process, ref_provider still has problem

File: gazebo/scout_gazebo/urdf/base.xacro (robot description, xacro)
@@ -47,5 +47,5 @@
     <xacro:include filename="$(find scout_gazebo)/urdf/laser_support.xacro" />
     <xacro:include filename="$(find velodyne_description)/urdf/VLP-16.urdf.xacro"/>
-    <xacro:VLP-16 parent="support" name="velodyne" topic="/velodyne_points" organize_cloud="${organize_cloud}" hz="10" samples="440" gpu="${gpu}">
+    <xacro:VLP-16 parent="support" name="velodyne" topic="/velodyne_points" organize_cloud="${organize_cloud}" hz="10" samples="1800" max_range="150" gpu="${gpu}">
           <origin xyz="0 0 ${support_length/2}" rpy="0 0 0" />
     </xacro:VLP-16>
@@ -53,5 +53,5 @@
     <xacro:include filename="$(find scout_gazebo)/urdf/imu.xacro"/>
     <xacro:imu sensor_name="imu" parent_link="base_link">
-    <origin rpy="0 0 0" xyz="-0.03 0 ${base_z_size/2}"/>
+    <origin rpy="0 0 0" xyz="0 0 0"/>
     </xacro:imu>
     <!-- 机器人导航控制模块 -->

File: gazebo/scout_gazebo/urdf/laser_support.xacro (robot description, xacro)
@@ -2,7 +2,7 @@
 <robot name="laser_support" xmlns:xacro="http://wiki.ros.org/xacro">
     <!-- 雷达支架 -->
-    <xacro:property name="support_length" value="3.00" /> <!-- 支架长度 -->
+    <xacro:property name="support_length" value="0.057" /> <!-- 支架长度 -->
     <xacro:property name="support_radius" value="0.025" /> <!-- 支架半径 -->
-    <xacro:property name="support_x_size" value="-0.2" /> <!-- 支架安装的x坐标 -->
+    <xacro:property name="support_x_size" value="0.0" /> <!-- 支架安装的x坐标 -->
     <xacro:property name="support_y_size" value="0.0" /> <!-- 支架安装的y坐标 -->
     <xacro:property name="support_z_size" value="${base_z_size/2+support_length/2}" /> <!-- 支架安装的z坐标:底盘高度 / 2 + 支架高度 / 2  -->

File: gazebo/scout_gazebo/urdf/move.xacro (robot description, xacro)
@@ -22,5 +22,5 @@
     <!-- 控制器 -->
     <gazebo>
-  		<plugin name="skid_steer_drive_controller" filename="libgazebo_ros_skid_steer_drive.so">
+  		<plugin name="skid_steer_drive_controller" filename="libgazebo_teleop_twist_keyboard.so">
     		<updateRate>100.0</updateRate>
     		<robotNamespace>/</robotNamespace>
@@ -35,4 +35,10 @@
     		<topicName>cmd_vel</topicName>
     		<broadcastTF>false</broadcastTF>
+    		<commandTopic>cmd_vel</commandTopic>
+    		<odometryTopic>odom</odometryTopic>
+    		<odometryFrame>odom</odometryFrame>
+				<covariance_x>0.0001</covariance_x>
+				<covariance_y>0.0001</covariance_y>
+				<covariance_yaw>0.0001</covariance_yaw>
   		</plugin>
 	</gazebo>
@@ -44,4 +50,5 @@
       <odometryRate>20.0</odometryRate>
       <robotBaseFrame>base_link</robotBaseFrame>
+			<cmdTimeout>-1.000</cmdTimeout>
     </plugin>
   </gazebo>

File: gazebo/scout_gazebo/urdf/plugin.xacro (robot description, xacro)
@@ -7,5 +7,5 @@
         <bodyName>base_link</bodyName>
         <topicName>base_pose_ground_truth</topicName>
-        <gaussianNoise>0.01</gaussianNoise>
+        <gaussianNoise>0</gaussianNoise>
         <frameName>map</frameName>
         <xyzOffsets>0 0 0</xyzOffsets>
